File: KiCad Designs With PCB/Exercise 2/Exercise 2.kicad_pcb (KiCad board)
At the start: 2 copper layers, 53.3 x 58.4 mm, 10 parts, among them J1 Conn_01x02_Male, U1 NE555D

Commit message: Gerber PCB Files added
Routing:
- net GND: track 80.0 -> 78.5 mm
